File: source/main.kicad_pcb (KiCad board)
At the start: 2 copper layers, 0 parts

Commit message: Revision 1.0.0 (#1)
---------

Co-authored-by: Ioannis P <ioannis@iteng.nl>
Parts:
- added C1: 100nF 16V X7R, lcsc:C0402, F.Cu at (74.1, 44.5)
- added D1: LED, lcsc:LED0402-R-RD_RED, F.Cu at (4.55, 20.6)
- added D10: LED, lcsc:LED0402-R-RD_RED, F.Cu at (16.7, 3.50)
- added D11: LED, lcsc:LED0402-R-RD_RED, F.Cu at (4.55, 17.8)
- added D12: LED, lcsc:LED0402-R-RD_RED, F.Cu at (4.55, 14.9)
- added D13: LED, lcsc:LED0402-R-RD_RED, F.Cu at (4.55, 12.1)
- added D14: LED, lcsc:LED0402-R-RD_RED, F.Cu at (4.55, 9.21)
- added D15: LED, lcsc:LED0402-R-RD_RED, F.Cu at (4.55, 6.36)
- added D16: LED, lcsc:LED0402-R-RD_RED, F.Cu at (4.55, 3.50)
- added D17: LED, lcsc:LED0402-R-RD_RED, F.Cu at (7.58, 9.21)
- added D18: LED, lcsc:LED0402-R-RD_RED, F.Cu at (26.2, 20.6)
- added D19: LED, lcsc:LED0402-R-RD_RED, F.Cu at (26.2, 17.8)
- added D2: LED, lcsc:LED0402-R-RD_RED, F.Cu at (16.7, 20.6)
- added D20: LED, lcsc:LED0402-R-RD_RED, F.Cu at (26.2, 14.9)
- added D21: LED, lcsc:LED0402-R-RD_RED, F.Cu at (26.2, 12.1)
- added D22: LED, lcsc:LED0402-R-RD_RED, F.Cu at (26.2, 9.21)
- added D23: LED, lcsc:LED0402-R-RD_RED, F.Cu at (26.2, 6.36)
- added D24: LED, lcsc:LED0402-R-RD_RED, F.Cu at (29.2, 9.21)
- added D25: LED, lcsc:LED0402-R-RD_RED, F.Cu at (32.3, 9.21)
- added D26: LED, lcsc:LED0402-R-RD_RED, F.Cu at (35.3, 9.21)
- added D27: LED, lcsc:LED0402-R-RD_RED, F.Cu at (38.3, 20.6)
- added D28: LED, lcsc:LED0402-R-RD_RED, F.Cu at (38.3, 17.8)
- added D29: LED, lcsc:LED0402-R-RD_RED, F.Cu at (38.3, 14.9)
- added D3: LED, lcsc:LED0402-R-RD_RED, F.Cu at (13.6, 9.21)
- added D30: LED, lcsc:LED0402-R-RD_RED, F.Cu at (38.3, 12.1)
- added D31: LED, lcsc:LED0402-R-RD_RED, F.Cu at (38.3, 9.21)
- added D32: LED, lcsc:LED0402-R-RD_RED, F.Cu at (38.3, 6.36)
- added D33: LED, lcsc:LED0402-R-RD_RED, F.Cu at (29.2, 3.50)
- added D34: LED, lcsc:LED0402-R-RD_RED, F.Cu at (32.3, 3.50)
- added D35: LED, lcsc:LED0402-R-RD_RED, F.Cu at (35.3, 3.50)
- added D36: LED, lcsc:LED0402-R-RD_RED, F.Cu at (50.9, 20.6)
- added D37: LED, lcsc:LED0402-R-RD_RED, F.Cu at (53.9, 20.6)
- added D38: LED, lcsc:LED0402-R-RD_RED, F.Cu at (57.0, 20.6)
- added D39: LED, lcsc:LED0402-R-RD_RED, F.Cu at (60.0, 17.8)
- added D4: LED, lcsc:LED0402-R-RD_RED, F.Cu at (10.6, 9.21)
- added D40: LED, lcsc:LED0402-R-RD_RED, F.Cu at (47.9, 17.8)
- added D41: LED, lcsc:LED0402-R-RD_RED, F.Cu at (47.9, 14.9)
- added D42: LED, lcsc:LED0402-R-RD_RED, F.Cu at (47.9, 12.1)
- added D43: LED, lcsc:LED0402-R-RD_RED, F.Cu at (47.9, 9.21)
- added D44: LED, lcsc:LED0402-R-RD_RED, F.Cu at (47.9, 6.36)
- added D45: LED, lcsc:LED0402-R-RD_RED, F.Cu at (60.0, 6.36)
- added D46: LED, lcsc:LED0402-R-RD_RED, F.Cu at (50.9, 3.50)
- added D47: LED, lcsc:LED0402-R-RD_RED, F.Cu at (53.9, 3.50)
- added D48: LED, lcsc:LED0402-R-RD_RED, F.Cu at (57.0, 3.50)
- added D49: LED, lcsc:LED0402-R-RD_RED, F.Cu at (81.7, 20.6)
- added D5: LED, lcsc:LED0402-R-RD_RED, F.Cu at (16.7, 17.8)
- added D50: LED, lcsc:LED0402-R-RD_RED, F.Cu at (81.7, 17.8)
- added D51: LED, lcsc:LED0402-R-RD_RED, F.Cu at (81.7, 14.9)
- added D52: LED, lcsc:LED0402-R-RD_RED, F.Cu at (78.6, 12.1)
- added D53: LED, lcsc:LED0402-R-RD_RED, F.Cu at (78.6, 6.36)
- added D54: LED, lcsc:LED0402-R-RD_RED, F.Cu at (69.5, 20.6)
- added D55: LED, lcsc:LED0402-R-RD_RED, F.Cu at (69.5, 17.8)
- added D56: LED, lcsc:LED0402-R-RD_RED, F.Cu at (69.5, 14.9)
- added D57: LED, lcsc:LED0402-R-RD_RED, F.Cu at (69.5, 12.1)
- added D58: LED, lcsc:LED0402-R-RD_RED, F.Cu at (69.5, 9.21)
- added D59: LED, lcsc:LED0402-R-RD_RED, F.Cu at (69.5, 6.36)
- added D6: LED, lcsc:LED0402-R-RD_RED, F.Cu at (16.7, 14.9)
- added D60: LED, lcsc:LED0402-R-RD_RED, F.Cu at (69.5, 3.50)
- added D61: LED, lcsc:LED0402-R-RD_RED, F.Cu at (72.6, 9.21)
- added D62: LED, lcsc:LED0402-R-RD_RED, F.Cu at (75.6, 9.21)
- added D63: LED, lcsc:LED0402-R-RD_RED, F.Cu at (81.7, 3.50)
- added D7: LED, lcsc:LED0402-R-RD_RED, F.Cu at (16.7, 12.1)
- added D8: LED, lcsc:LED0402-R-RD_RED, F.Cu at (16.7, 9.21)
- added D9: LED, lcsc:LED0402-R-RD_RED, F.Cu at (16.7, 6.36)
- added F1: Fuse, lcsc:F0402, F.Cu at (76.3, 42.0)
- added LOGO1: Faebryk_Logo, logo:faebryk_logo, F.Cu at (42.8, 48.0)
- added P1: USB_Type_C_Receptacle_16_pin, lcsc:USB-C-SMD_TYPE-C-6PIN-2MD-073, F.Cu at (81.1, 44.5)
- added R1: 100Ω, lcsc:R0402, F.Cu at (5.65, 20.4)
- added R10: 100Ω, lcsc:R0402, F.Cu at (17.8, 3.25)
- added R11: 100Ω, lcsc:R0402, F.Cu at (5.65, 17.5)
- added R12: 100Ω, lcsc:R0402, F.Cu at (5.65, 14.7)
- added R13: 100Ω, lcsc:R0402, F.Cu at (5.65, 11.8)
- added R14: 100Ω, lcsc:R0402, F.Cu at (5.65, 8.96)
- added R15: 100Ω, lcsc:R0402, F.Cu at (5.65, 6.11)
- added R16: 100Ω, lcsc:R0402, F.Cu at (5.65, 3.25)
- added R17: 100Ω, lcsc:R0402, F.Cu at (8.68, 8.96)
- added R18: 100Ω, lcsc:R0402, F.Cu at (27.3, 20.4)
- added R19: 100Ω, lcsc:R0402, F.Cu at (27.3, 17.5)
- added R2: 100Ω, lcsc:R0402, F.Cu at (17.8, 20.4)
- added R20: 5.1kΩ, lcsc:R0402, F.Cu at (76.3, 45.8)
- added R21: 5.1kΩ, lcsc:R0402, F.Cu at (76.3, 43.2)
- added R22: 100Ω, lcsc:R0402, F.Cu at (27.3, 14.7)
- added R23: 100Ω, lcsc:R0402, F.Cu at (27.3, 11.8)
- added R24: 100Ω, lcsc:R0402, F.Cu at (27.3, 8.96)
- added R25: 100Ω, lcsc:R0402, F.Cu at (27.3, 6.11)
- added R26: 100Ω, lcsc:R0402, F.Cu at (30.3, 8.96)
- added R27: 100Ω, lcsc:R0402, F.Cu at (33.4, 8.96)
- added R28: 100Ω, lcsc:R0402, F.Cu at (36.4, 8.96)
- added R29: 100Ω, lcsc:R0402, F.Cu at (39.4, 20.4)
- added R3: 100Ω, lcsc:R0402, F.Cu at (14.7, 8.96)
- added R30: 100Ω, lcsc:R0402, F.Cu at (39.4, 17.5)
- added R31: 100Ω, lcsc:R0402, F.Cu at (39.4, 14.7)
- added R32: 100Ω, lcsc:R0402, F.Cu at (39.4, 11.8)
- added R33: 100Ω, lcsc:R0402, F.Cu at (39.4, 8.96)
- added R34: 100Ω, lcsc:R0402, F.Cu at (39.4, 6.11)
- added R35: 100Ω, lcsc:R0402, F.Cu at (30.3, 3.25)
- added R36: 100Ω, lcsc:R0402, F.Cu at (33.4, 3.25)
- added R37: 100Ω, lcsc:R0402, F.Cu at (36.4, 3.25)
- added R38: 100Ω, lcsc:R0402, F.Cu at (52.0, 20.4)
- added R39: 100Ω, lcsc:R0402, F.Cu at (55.0, 20.4)
- added R4: 100Ω, lcsc:R0402, F.Cu at (11.7, 8.96)
- added R40: 100Ω, lcsc:R0402, F.Cu at (58.1, 20.4)
- added R41: 100Ω, lcsc:R0402, F.Cu at (61.1, 17.5)
- added R42: 100Ω, lcsc:R0402, F.Cu at (49.0, 17.5)
- added R43: 100Ω, lcsc:R0402, F.Cu at (49.0, 14.7)
- added R44: 100Ω, lcsc:R0402, F.Cu at (49.0, 11.8)
- added R45: 100Ω, lcsc:R0402, F.Cu at (49.0, 8.96)
- added R46: 100Ω, lcsc:R0402, F.Cu at (49.0, 6.11)
- added R47: 100Ω, lcsc:R0402, F.Cu at (61.1, 6.11)
- added R48: 100Ω, lcsc:R0402, F.Cu at (52.0, 3.25)
- added R49: 100Ω, lcsc:R0402, F.Cu at (55.0, 3.25)
- added R5: 100Ω, lcsc:R0402, F.Cu at (17.8, 17.5)
- added R50: 100Ω, lcsc:R0402, F.Cu at (58.1, 3.25)
- added R51: 100Ω, lcsc:R0402, F.Cu at (82.8, 20.4)
- added R52: 100Ω, lcsc:R0402, F.Cu at (82.8, 17.5)
- added R53: 100Ω, lcsc:R0402, F.Cu at (82.8, 14.7)
- added R54: 100Ω, lcsc:R0402, F.Cu at (79.7, 11.8)
- added R55: 100Ω, lcsc:R0402, F.Cu at (79.7, 6.11)
- added R56: 100Ω, lcsc:R0402, F.Cu at (70.6, 20.4)
- added R57: 100Ω, lcsc:R0402, F.Cu at (70.6, 17.5)
- added R58: 100Ω, lcsc:R0402, F.Cu at (70.6, 14.7)
- added R59: 100Ω, lcsc:R0402, F.Cu at (70.6, 11.8)
- added R6: 100Ω, lcsc:R0402, F.Cu at (17.8, 14.7)
- added R60: 100Ω, lcsc:R0402, F.Cu at (70.6, 8.96)
- added R61: 100Ω, lcsc:R0402, F.Cu at (70.6, 6.11)
- added R62: 100Ω, lcsc:R0402, F.Cu at (70.6, 3.25)
- added R63: 100Ω, lcsc:R0402, F.Cu at (73.7, 8.96)
- added R64: 100Ω, lcsc:R0402, F.Cu at (76.7, 8.96)
- added R65: 100Ω, lcsc:R0402, F.Cu at (82.8, 3.25)
- added R7: 100Ω, lcsc:R0402, F.Cu at (17.8, 11.8)
- added R8: 100Ω, lcsc:R0402, F.Cu at (17.8, 8.96)
- added R9: 100Ω, lcsc:R0402, F.Cu at (17.8, 6.11)
Routing:
- net P1-9-R21-1: track 0.00 -> 1.94 mm
- net P1-4-R20-1: track 0.00 -> 1.94 mm
- net vbus: track 0.00 -> 1.71 mm, vias 0 -> 2
- net D55-1-R57-1: track 0.00 -> 1.10 mm
- net D61-1-R63-1: track 0.00 -> 1.10 mm
- net D60-1-R62-1: track 0.00 -> 1.10 mm
- net D59-1-R61-1: track 0.00 -> 1.10 mm
- net D58-1-R60-1: track 0.00 -> 1.10 mm
- net D57-1-R59-1: track 0.00 -> 1.10 mm
- net D56-1-R58-1: track 0.00 -> 1.10 mm
- net D54-1-R56-1: track 0.00 -> 1.10 mm
- net D39-1-R41-1: track 0.00 -> 1.10 mm
- net D28-1-R30-1: track 0.00 -> 1.10 mm
- net D48-1-R50-1: track 0.00 -> 1.10 mm
- net D47-1-R49-1: track 0.00 -> 1.10 mm
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- added copper zone on F.Cu, net gnd
- added copper zone on B.Cu, net vbus
Other:
- board outline added: 85.6 x 54 mm
- board text added: "Name: Hat Black"
- board text added: "RPI PINOUT"
- board text added: "Tel: +31 6 42069666"
- board text added: "Url: github.com/faebryk"

Commit message: Improve routing & Enable artifacts & Improve font (#2)
* Improve routing

* Layout: improve font rendering

Use updated FontLayout
Group font settings in app.py
Render silk zones for text polygons

* Enable artifacts
* Remove actual artifacts
* Use newest app lib in faebryk
* Adjust font parameters

---------

Co-authored-by: Jasper Smit <git@jrhrsmit.nl>
Parts:
- removed D50, D51, D52, D53, D54, D55, D56, D57, D58, D59, D60, D61, D62, D63: LED, lcsc:LED0402-R-RD_RED
- removed R52, R53, R54, R55, R56, R57, R58, R59, R60, R61, R62, R63, R64, R65: 100Ω, lcsc:R0402
- moved D49 26.4 mm to (60.2, 5.25)
- moved R51 26.4 mm to (61.4, 5.00)
- moved D27 21.5 mm to (23.4, 5.25)
- moved R29 21.5 mm to (24.5, 5.00)
- moved D36 19.9 mm to (38.4, 5.25)
- moved R38 19.9 mm to (39.5, 5.00)
- moved D37 19.4 mm to (42.1, 5.25)
- moved R39 19.4 mm to (43.2, 5.00)
- moved D45 16.6 mm to (50.2, 19.8)
- moved R47 16.6 mm to (51.3, 19.5)
- moved D33 15.2 mm to (35.2, 17.4)
- moved R35 15.2 mm to (36.4, 17.2)
- moved D5 13.6 mm to (30.2, 16.9)
- moved R5 13.6 mm to (31.3, 16.7)
- moved D13 13.3 mm to (15.3, 20.0)
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Connections:
- D1 pad 2: D1-2 -> vbus
- D10 pad 2: D10-2 -> vbus
- D11 pad 2: D11-2 -> vbus
- D12 pad 2: D12-2 -> vbus
- D13 pad 2: D13-2 -> vbus
- D14 pad 2: D14-2 -> vbus
- D15 pad 2: D15-2 -> vbus
- D16 pad 2: D16-2 -> vbus
- D17 pad 2: D17-2 -> vbus
- D18 pad 2: D18-2 -> vbus
- D19 pad 2: D19-2 -> vbus
- D2 pad 2: D2-2 -> vbus
- D20 pad 2: D20-2 -> vbus
- D21 pad 2: D21-2 -> vbus
- D22 pad 2: D22-2 -> vbus
- D23 pad 2: D23-2 -> vbus
- D24 pad 2: D24-2 -> vbus
- D25 pad 2: D25-2 -> vbus
- D26 pad 2: D26-2 -> vbus
- D27 pad 2: D27-2 -> vbus
- D28 pad 2: D28-2 -> vbus
- D29 pad 2: D29-2 -> vbus
- D3 pad 2: D3-2 -> vbus
- D30 pad 2: D30-2 -> vbus
- D31 pad 2: D31-2 -> vbus
- D32 pad 2: D32-2 -> vbus
- D33 pad 2: D33-2 -> vbus
- D34 pad 2: D34-2 -> vbus
- D35 pad 2: D35-2 -> vbus
- D36 pad 2: D36-2 -> vbus
- D37 pad 2: D37-2 -> vbus
- D38 pad 2: D38-2 -> vbus
- D39 pad 2: D39-2 -> vbus
- D4 pad 2: D4-2 -> vbus
- D40 pad 2: D40-2 -> vbus
- D41 pad 2: D41-2 -> vbus
- D42 pad 2: D42-2 -> vbus
- D43 pad 2: D43-2 -> vbus
- D44 pad 2: D44-2 -> vbus
- D45 pad 2: D45-2 -> vbus
- D46 pad 2: D46-2 -> vbus
- D47 pad 2: D47-2 -> vbus
- D48 pad 2: D48-2 -> vbus
- D49 pad 2: D49-2 -> vbus
- D5 pad 2: D5-2 -> vbus
- D6 pad 2: D6-2 -> vbus
- D7 pad 2: D7-2 -> vbus
- D8 pad 2: D8-2 -> vbus
- D9 pad 2: D9-2 -> vbus
- R1 pad 2: R1-2 -> gnd
- R10 pad 2: R10-2 -> gnd
- R11 pad 2: R11-2 -> gnd
- R12 pad 2: R12-2 -> gnd
- R13 pad 2: R13-2 -> gnd
- R14 pad 2: R14-2 -> gnd
- R15 pad 2: R15-2 -> gnd
- R16 pad 2: R16-2 -> gnd
- R17 pad 2: R17-2 -> gnd
- R18 pad 2: R18-2 -> gnd
- R19 pad 2: R19-2 -> gnd
- R2 pad 2: R2-2 -> gnd
- R22 pad 2: R22-2 -> gnd
- R23 pad 2: R23-2 -> gnd
- R24 pad 2: R24-2 -> gnd
- R25 pad 2: R25-2 -> gnd
- R26 pad 2: R26-2 -> gnd
- R27 pad 2: R27-2 -> gnd
- R28 pad 2: R28-2 -> gnd
- R29 pad 2: R29-2 -> gnd
- R3 pad 2: R3-2 -> gnd
- R30 pad 2: R30-2 -> gnd
- R31 pad 2: R31-2 -> gnd
- R32 pad 2: R32-2 -> gnd
- R33 pad 2: R33-2 -> gnd
- R34 pad 2: R34-2 -> gnd
- R35 pad 2: R35-2 -> gnd
- R36 pad 2: R36-2 -> gnd
- R37 pad 2: R37-2 -> gnd
- R38 pad 2: R38-2 -> gnd
- R39 pad 2: R39-2 -> gnd
- R4 pad 2: R4-2 -> gnd
- R40 pad 2: R40-2 -> gnd
- R41 pad 2: R41-2 -> gnd
- R42 pad 2: R42-2 -> gnd
- R43 pad 2: R43-2 -> gnd
- R44 pad 2: R44-2 -> gnd
- R45 pad 2: R45-2 -> gnd
- R46 pad 2: R46-2 -> gnd
- R47 pad 2: R47-2 -> gnd
- R48 pad 2: R48-2 -> gnd
- R49 pad 2: R49-2 -> gnd
- R5 pad 2: R5-2 -> gnd
- R50 pad 2: R50-2 -> gnd
- R51 pad 2: R51-2 -> gnd
- R6 pad 2: R6-2 -> gnd
- R7 pad 2: R7-2 -> gnd
- R8 pad 2: R8-2 -> gnd
- R9 pad 2: R9-2 -> gnd
Routing:
- net vbus: track 1.71 -> 45.5 mm, vias 2 -> 50
- net F1-1-P1-11-P1-2: track 0.00 -> 8.53 mm
- net D55-1-R57-1: track 1.10 -> 0.00 mm
- net D61-1-R63-1: track 1.10 -> 0.00 mm
- net D60-1-R62-1: track 1.10 -> 0.00 mm
- net D59-1-R61-1: track 1.10 -> 0.00 mm
- net D58-1-R60-1: track 1.10 -> 0.00 mm
- net D57-1-R59-1: track 1.10 -> 0.00 mm
- net D56-1-R58-1: track 1.10 -> 0.00 mm
- net D54-1-R56-1: track 1.10 -> 0.00 mm
- net D50-1-R52-1: track 1.10 -> 0.00 mm
- net D63-1-R65-1: track 1.10 -> 0.00 mm
- net D62-1-R64-1: track 1.10 -> 0.00 mm
- net D53-1-R55-1: track 1.10 -> 0.00 mm
- net D52-1-R54-1: track 1.10 -> 0.00 mm
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Other:
- board text removed: "RPI PINOUT"
